Commit message: added code for the 4 wheeler model and launch file

File: src/simple4wheeler/model/simple4wheeler.xacro (robot description, xacro)
@@ -1,3 +1,4 @@
 <robot name="simple4wheeler" xmlns:xacro="http://www.ros.org/wiki/xacro">
+    <xacro:property name="pii" value="3.14159265359"/>
     <link name="map">
     </link>
@@ -30,8 +31,9 @@
         <child link="link_chassis"/>
     </joint>
+    <!-- Existing Wheel -->
     <link name="link_right_back_wheel">
         <inertial>
             <mass value="0.2"/>
-            <origin xyz="0.075 0.17 -0.03" rpy="1.5708 1.5708 0"/>
+            <origin xyz="0.075 -0.17 -0.03" rpy="1.5708 1.5708 0"/>
             <inertia ixx="0.00052"
                      ixy="0"
@@ -53,5 +55,5 @@
     </link>
     <joint name="joint_right_back_wheel" type="continuous">
-        <origin xyz="0.075 0.17 -0.03" rpy="0 1.5708 1"/>
+        <origin xyz="0.075 -0.17 -0.03" rpy="0 1.5708 1"/>
         <parent link="link_chassis"/>
         <child link="link_right_back_wheel"/>
@@ -60,4 +62,41 @@
         <joint_properties damping="1.0" friction="1.0"/>
     </joint>
+    <!-- Additional Wheels -->
+    <xacro:macro name="wheel" params="prefix x y z">
+        <link name="$(prefix)_wheel">
+            <inertial>
+                <mass value="0.2"/>
+                <origin xyz="$(x) $(y) $(z)" rpy="1.5708 1.5708 0"/>
+                <inertia ixx="0.00052"
+                         ixy="0"
+                         ixz="0"
+                         iyy="0.00052"
+                         iyz="0"
+                         izz="0.00100"/>
+            </inertial>
+            <collision name="collision_$(prefix)_wheel">
+                <geometry>
+                    <cylinder radius="0.1" length="0.04"/>
+                </geometry>
+            </collision>
+            <visual name="visual_$(prefix)_wheel">
+                <geometry>
+                    <cylinder radius="0.1" length="0.04"/>
+                </geometry>
+            </visual>
+        </link>
+        <joint name="joint_$(prefix)_wheel" type="continuous">
+            <origin xyz="$(x) $(y) $(z)" rpy="0 1.5708 1"/>
+            <parent link="link_chassis"/>
+            <child link="$(prefix)_wheel"/>
+            <axis rpy="0 0 0" xyz="1 0 0"/>
+            <limit effort="10" velocity="10"/>
+            <joint_properties damping="1.0" friction="1.0"/>
+        </joint>
+    </xacro:macro>
+    <xacro:wheel prefix="front_right" x="0.25" y="0.15" z="-0.03"/>
+    <xacro:wheel prefix="front_left" x="0.25" y="-0.15" z="-0.03"/>
+    <xacro:wheel prefix="back_left" x="-0.25" y="-0.15" z="-0.03"/>
+    <xacro:wheel prefix="back_right" x="-0.25" y="0.15" z="-0.03"/>
     <link name="link_lidar">
         <inertial>
@@ -119,3 +158,58 @@
         </sensor>
     </gazebo>
+    <gazebo>
+        <plugin name="skid_steer_drive_controller" filename="libgazebo_ros_skid_steer_drive.so">
+            <updateRate>100.0</updateRate>
+            <robotNamespace>/</robotNamespace>
+            <leftFrontJoint>front_left_wheel_joint</leftFrontJoint>
+            <rightFrontJoint>front_right_wheel_joint</rightFrontJoint>
+            <leftRearJoint>back_left_wheel_joint</leftRearJoint>
+            <rightRearJoint>back_right_wheel_joint</rightRearJoint>
+            <wheelSeparation>0.4</wheelSeparation>
+            <wheelDiameter>0.215</wheelDiameter>
+            <robotBaseFrame>base_link</robotBaseFrame>
+            <torque>20</torque>
+            <topicName>cmd_vel</topicName>
+            <broadcastTF>false</broadcastTF>
+        </plugin>
+    </gazebo>
+    <gazebo reference="link_ultra_sonic1">
+        <sensor type="ray" name="sensor_sonic1">
+            <pose> 0 0 0 0 0 0</pose>
+            <update_rate>60</update_rate>
+            <visualize>true</visualize>
+            <ray>
+                <scan>
+                    <horizontal>
+                        <samples>5</samples>
+                        <resolution>1</resolution>
+                        <min_angle>-0.05</min_angle>
+                        <max_angle>0.05</max_angle>
+                    </horizontal>
+                    <vertical>
+                        <samples>1</samples>
+                        <resolution>1</resolution>
+                        <min_angle>-0.05</min_angle>
+                        <max_angle>0.05</max_angle>
+                    </vertical>
+                </scan>
+                <range>
+                    <min>0.01</min>
+                    <max>10</max>
+                    <resolution>0.01</resolution>
+                </range>
+            </ray>
+            <plugin name="controller_sonic1" filename="libgazebo_ros_range.so">
+                <gaussianNoise>0.005</gaussianNoise>
+                <alwaysOn>true</alwaysOn>
+                <updateRate>60</updateRate>
+                <topicName>/ultrasonic1</topicName>
+                <frameName>link_ultra_sonic1</frameName>
+                <minRange>0.01</minRange>
+                <maxRange>10</maxRange>
+                <fov>0.5</fov>
+                <radiation>ultrasound</radiation>
+            </plugin>
+        </sensor>
+    </gazebo>
 </robot>

Commit message: commit1

File: src/simple4wheeler/model/simple4wheeler.xacro (robot description, xacro)
@@ -1,18 +1,17 @@
 <robot name="simple4wheeler" xmlns:xacro="http://www.ros.org/wiki/xacro">
-    <xacro:property name="pii" value="3.14159265359"/>
     <link name="map">
     </link>
     <link name="link_chassis">
-        <!-- pose x,y,z, roll, pitch, yaw -->
-        <pose>0 0 0.1 0 0 0</pose>
-        <inertial>
-            <mass value="5"/>
+        <!--pose x,y,z, roll, pitch, yaw-->
+        <pose> 0 0 0.1 0 0 0 </pose>
+        <inertial>
+            <mass value="100"/>
             <origin rpy="0 0 0" xyz="0 0 0.1"/>
-            <inertia ixx="0.03954"
-                     ixy="0"
-                     ixz="0"
-                     iyy="0.10620"
-                     iyz="0"
-                     izz="0.10620"/>
+            <inertia   ixx="0.03954"
+                        ixy="0.0"
+                        ixz="0.0"
+                        iyy="0.10620"
+                        iyz="0.0"
+                        izz="0.10620"/>
         </inertial>
         <collision name="collision_chassis">
@@ -31,81 +30,133 @@
         <child link="link_chassis"/>
     </joint>
-    <!-- Existing Wheel -->
-    <link name="link_right_back_wheel">
-        <inertial>
-            <mass value="0.2"/>
-            <origin xyz="0.075 -0.17 -0.03" rpy="1.5708 1.5708 0"/>
-            <inertia ixx="0.00052"
-                     ixy="0"
-                     ixz="0"
-                     iyy="0.00052"
-                     iyz="0"
-                     izz="0.00100"/>
-        </inertial>
-        <collision name="collision_right_back_wheel">
-            <geometry>
-                <cylinder radius="0.1" length="0.04"/>
-            </geometry>
-        </collision>
-        <visual name="visual_right_back_wheel">
-            <geometry>
-                <cylinder radius="0.1" length="0.04"/>
-            </geometry>
-        </visual>
-    </link>
-    <joint name="joint_right_back_wheel" type="continuous">
-        <origin xyz="0.075 -0.17 -0.03" rpy="0 1.5708 1"/>
-        <parent link="link_chassis"/>
-        <child link="link_right_back_wheel"/>
-        <axis rpy="0 0 0" xyz="1 0 0"/>
-        <limit effort="10" velocity="10"/>
-        <joint_properties damping="1.0" friction="1.0"/>
-    </joint>
-    <!-- Additional Wheels -->
-    <xacro:macro name="wheel" params="prefix x y z">
-        <link name="$(prefix)_wheel">
-            <inertial>
-                <mass value="0.2"/>
-                <origin xyz="$(x) $(y) $(z)" rpy="1.5708 1.5708 0"/>
-                <inertia ixx="0.00052"
-                         ixy="0"
-                         ixz="0"
-                         iyy="0.00052"
-                         iyz="0"
-                         izz="0.00100"/>
-            </inertial>
-            <collision name="collision_$(prefix)_wheel">
-                <geometry>
-                    <cylinder radius="0.1" length="0.04"/>
-                </geometry>
-            </collision>
-            <visual name="visual_$(prefix)_wheel">
-                <geometry>
-                    <cylinder radius="0.1" length="0.04"/>
-                </geometry>
-            </visual>
-        </link>
-        <joint name="joint_$(prefix)_wheel" type="continuous">
-            <origin xyz="$(x) $(y) $(z)" rpy="0 1.5708 1"/>
-            <parent link="link_chassis"/>
-            <child link="$(prefix)_wheel"/>
-            <axis rpy="0 0 0" xyz="1 0 0"/>
-            <limit effort="10" velocity="10"/>
-            <joint_properties damping="1.0" friction="1.0"/>
-        </joint>
-    </xacro:macro>
-    <xacro:wheel prefix="front_right" x="0.25" y="0.15" z="-0.03"/>
-    <xacro:wheel prefix="front_left" x="0.25" y="-0.15" z="-0.03"/>
-    <xacro:wheel prefix="back_left" x="-0.25" y="-0.15" z="-0.03"/>
-    <xacro:wheel prefix="back_right" x="-0.25" y="0.15" z="-0.03"/>
-    <link name="link_lidar">
+   <link name = "link_right_back_wheel">
+        <inertial>
+            <mass value = "5"/>
+            <origin rpy = "0 0 0" xyz = "0 0 0.1"/>
+            <inertia ixx = "0.03954"
+                 ixy = "0"
+                 ixz = "0"
+                 iyy = "0.10620"
+                 iyz = "0"
+                 izz = "0.10620"/>
+        </inertial>
+        <collision name = "collision_right_back_wheel">
+            <geometry>
+                <cylinder length = "0.04" radius = "0.1"/>
+            </geometry>
+        </collision>
+        <visual name = "visual_right_back_wheel">
+            <geometry>
+                <cylinder length = "0.04" radius = "0.1"/>
+            </geometry>
+        </visual>
+    </link>
+    <joint name = "joint_right_back_wheel" type = "continuous">
+        <origin rpy = "1.57 1.57 0" xyz = "-0.18 0.15 0"/>
+        <parent link = "link_chassis"/>
+        <child link = "link_right_back_wheel"/>
+        <axis rpy = "0 0 0" xyz = "0 0 1"/>
+        <limit effort = "10" velocity = "10"/>
+        <joint_properties damping = "1.0" friction = "1.0"/>
+    </joint>
+    <link name = "link_left_back_wheel">
+        <inertial>
+            <mass value = "5"/>
+            <origin rpy = "0 0 0" xyz = "0 0 0.1"/>
+            <inertia ixx = "0.03954"
+                 ixy = "0"
+                 ixz = "0"
+                 iyy = "0.10620"
+                 iyz = "0"
+                 izz = "0.10620"/>
+        </inertial>
+        <collision name = "collision_left_back_wheel">
+            <geometry>
+                <cylinder length = "0.04" radius = "0.1"/>
+            </geometry>
+        </collision>
+        <visual name = "visual_left_back_wheel">
+            <geometry>
+                <cylinder length = "0.04" radius = "0.1"/>
+            </geometry>
+        </visual>
+    </link>
+    <joint name = "joint_left_back_wheel" type = "continuous">
+        <origin rpy = "1.57 1.57 0" xyz = "-0.18 -0.15 0"/>
+        <parent link = "link_chassis"/>
+        <child link = "link_left_back_wheel"/>
+        <axis rpy = "0 0 0" xyz = "0 0 1"/>
+        <limit effort = "10" velocity = "10"/>
+        <joint_properties damping = "1.0" friction = "1.0"/>
+    </joint>
+<link name = "link_right_front_wheel">
+        <inertial>
+            <mass value = "5"/>
+            <origin rpy = "0 0 0" xyz = "0 0 0.1"/>
+            <inertia ixx = "0.03954"
+                 ixy = "0"
+                 ixz = "0"
+                 iyy = "0.10620"
+                 iyz = "0"
+                 izz = "0.10620"/>
+        </inertial>
+        <collision name = "collision_right_front_wheel">
+            <geometry>
+                <cylinder length = "0.04" radius = "0.1"/>
+            </geometry>
+        </collision>
+        <visual name = "visual_right_front_wheel">
+            <geometry>
+                <cylinder length = "0.04" radius = "0.1"/>
+            </geometry>
+        </visual>
+    </link>
+    <joint name = "joint_right_front_wheel" type = "continuous">
+        <origin rpy = "1.57 1.57 0" xyz = "0.18 0.15 0"/>
+        <parent link = "link_chassis"/>
+        <child link = "link_right_front_wheel"/>
+        <axis rpy = "0 0 0" xyz = "0 0 1"/>
+        <limit effort = "10" velocity = "10"/>
+        <joint_properties damping = "1.0" friction = "1.0"/>
+    </joint>
+    <link name = "link_left_front_wheel">
+        <inertial>
+            <mass value = "5"/>
+            <origin rpy = "0 0 0" xyz = "0 0 0.1"/>
+            <inertia ixx = "0.03954"
+                 ixy = "0"
+                 ixz = "0"
+                 iyy = "0.10620"
+                 iyz = "0"
+                 izz = "0.10620"/>
+        </inertial>
+        <collision name = "collision_left_front_wheel">
+            <geometry>
+                <cylinder length = "0.04" radius = "0.1"/>
+            </geometry>
+        </collision>
+        <visual name = "visual_left_front_wheel">
+            <geometry>
+                <cylinder length = "0.04" radius = "0.1"/>
+            </geometry>
+        </visual>
+    </link>
+    <joint name = "joint_left_front_wheel" type = "continuous">
+        <origin rpy = "1.57 1.57 0" xyz = "0.18 -0.15 0"/>
+        <parent link = "link_chassis"/>
+        <child link = "link_left_front_wheel"/>
+        <axis rpy = "0 0 0" xyz = "0 0 1"/>
+        <limit effort = "10" velocity = "10"/>
+        <joint_properties damping = "1.0" friction = "1.0"/>
+    </joint>
+   <link name="link_lidar">
         <inertial>
             <mass value="0.05"/>
-            <inertia ixx="0.00001"
-                     ixy="0"
-                     ixz="0"
-                     iyy="0.00001"
-                     iyz="0"
-                     izz="0.00001"/>
+            <inertia    ixx="0.00001"
+                        ixy="0"
+                        ixz="0"
+                        iyy="0.00001"
+                        iyz="0"
+                        izz="0.00001"/>
         </inertial>
         <visual>
@@ -119,12 +170,12 @@
             </geometry>
         </collision>
-    </link>
+   </link>
     <joint name="joint_lidar" type="fixed">
-        <origin xyz="0 0 0.07" rpy="0 0 0"/>
+        <origin rpy="0 0 0" xyz="0 0 0.07" />
         <parent link="link_chassis"/>
         <child link="link_lidar"/>
     </joint>
     <gazebo reference="link_lidar">
-        <sensor type="ray" name="sensor_lidar">
+        <sensor name="sensor_lidar" type="ray">
             <update_rate>10</update_rate>
             <visualize>true</visualize>
@@ -144,5 +195,5 @@
                 <range>
                     <min>0.15</min>
-                    <max>3.5</max>
+                    <max>12</max>
                     <resolution>0.01</resolution>
                 </range>
@@ -158,36 +209,38 @@
         </sensor>
     </gazebo>
-    <gazebo>
-        <plugin name="skid_steer_drive_controller" filename="libgazebo_ros_skid_steer_drive.so">
-            <updateRate>100.0</updateRate>
-            <robotNamespace>/</robotNamespace>
-            <leftFrontJoint>front_left_wheel_joint</leftFrontJoint>
-            <rightFrontJoint>front_right_wheel_joint</rightFrontJoint>
-            <leftRearJoint>back_left_wheel_joint</leftRearJoint>
-            <rightRearJoint>back_right_wheel_joint</rightRearJoint>
-            <wheelSeparation>0.4</wheelSeparation>
-            <wheelDiameter>0.215</wheelDiameter>
-            <robotBaseFrame>base_link</robotBaseFrame>
-            <torque>20</torque>
-            <topicName>cmd_vel</topicName>
-            <broadcastTF>false</broadcastTF>
-        </plugin>
-    </gazebo>
-    <gazebo reference="link_ultra_sonic1">
-        <sensor type="ray" name="sensor_sonic1">
-            <pose> 0 0 0 0 0 0</pose>
-            <update_rate>60</update_rate>
+    <link name="link_ultrasonic">
+        <inertial>
+            <mass value="0.01"/>
+            <inertia ixx="0.00001" ixy="0" ixz="0" iyy="0.00001" iyz="0" izz="0.00001"/>
+        </inertial>
+        <visual>
+            <geometry>
+                <box size="0.017 0.07 0.03"/>
+            </geometry>
+        </visual>
+        <collision>
+            <geometry>
+                <box size="0.02 0.08 0.05"/>
+            </geometry>
+        </collision>
+    </link>
+    <joint name="joint_ultrasonic" type="fixed">
+        <origin rpy="0 0 0" xyz="0.22 0.07 0.058" />
+        <parent link="link_chassis"/>
+        <child link="link_ultrasonic"/>
+    </joint>
+    <gazebo reference="link_ultrasonic">
+        <sensor name="ultrasonic" type="ray">
+            <update_rate>10</update_rate>
             <visualize>true</visualize>
             <ray>
                 <scan>
                     <horizontal>
-                        <samples>5</samples>
-                        <resolution>1</resolution>
-                        <min_angle>-0.05</min_angle>
-                        <max_angle>0.05</max_angle>
+                        <samples>400</samples>
+                        <min_angle>-0.25</min_angle>
+                        <max_angle>0.2</max_angle>
                     </horizontal>
                     <vertical>
                         <samples>1</samples>
-                        <resolution>1</resolution>
                         <min_angle>-0.05</min_angle>
                         <max_angle>0.05</max_angle>
@@ -195,21 +248,80 @@
                 </scan>
                 <range>
-                    <min>0.01</min>
-                    <max>10</max>
+                    <min>0.15</min>
+                    <max>12</max>
                     <resolution>0.01</resolution>
                 </range>
             </ray>
-            <plugin name="controller_sonic1" filename="libgazebo_ros_range.so">
-                <gaussianNoise>0.005</gaussianNoise>
-                <alwaysOn>true</alwaysOn>
-                <updateRate>60</updateRate>
-                <topicName>/ultrasonic1</topicName>
-                <frameName>link_ultra_sonic1</frameName>
-                <minRange>0.01</minRange>
-                <maxRange>10</maxRange>
-                <fov>0.5</fov>
-                <radiation>ultrasound</radiation>
+            <plugin name="gazebo_ros_ultrasonic" filename="libgazebo_ros_range.so">
+                <gaussianNoise>0.01</gaussianNoise>
+                <updateRate>10</updateRate>
+                <topicName>ultrasonic</topicName>
+                <minRange>0.15</minRange>
+                <maxRange>14</maxRange>
+                <frameName>link_ultrasonic</frameName>
             </plugin>
         </sensor>
     </gazebo>
+    <link name="link_camera">
+        <inertial>
+            <mass value="0.01"/>
+            <inertia ixx="0.00001" ixy="0" ixz="0" iyy="0.00001" iyz="0" izz="0.00001"/>
+        </inertial>
+        <visual>
+            <geometry>
+                <box size="0.03 0.03 0.02"/>
+            </geometry>
+        </visual>
+        <collision>
+            <geometry>
+                <box size="0.032 0.032 0.04"/>
+            </geometry>
+        </collision>
+    </link>
+    <joint name="joint_camera" type="fixed">
+        <origin rpy="0 0 0" xyz="0.21 0 0.06" />
+        <parent link="link_chassis"/>
+        <child link="link_camera"/>
+    </joint>
+    <gazebo reference="link_camera">
+  <sensor type="camera" name="camera_sensor">
+    <update_rate>30.0</update_rate>
+    <camera name="head_camera">
+      <horizontal_fov>1.3962634</horizontal_fov>
+      <image>
+        <width>800</width>
+        <height>800</height>
+        <format>R8G8B8</format>
+      </image>
+      <clip>
+        <near>0.02</near>
+        <far>300</far>
+      </clip>
+    </camera>
+    <plugin name="camera_controller" filename="libgazebo_ros_camera.so">
+      <gaussianNoise>0.01</gaussianNoise>
+    <updateRate>10</updateRate>
+    <topicName>camera_image</topicName>
+    <minRange>0.15</minRange>
+    <maxRange>12</maxRange>
+    <frameName>link_camera</frameName>
+    </plugin>
+  </sensor>
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